File: schematics/spider_dropper/spider_dropper.kicad_pcb (KiCad board)
At the start: 2 copper layers, 80 x 20 mm, 10 parts, among them J1 12V DC, J2 JST_XH_3, J3 JST_XH_2, Q1 IRLZ34N, SW1 ZX40E20C01

Commit message: Checkpoint latest version of Rev D schematic and PCB.
Parts:
- moved Q1 1.14 mm to (143.1, 108.2)
Routing:
- net /MOTOR-: track 57.2 -> 56.3 mm
Changed lines of the file:
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@@
 	(title_block
 		(title "Slightly Smarter Simple Spider Dropper")
-		(date "2025-08-27")
+		(date "2025-08-28")
 		(rev "D")
 		(company "Adrian McCarthy")
@@
 	(footprint "Package_TO_SOT_THT:TO-220-3_Horizontal_TabDown"
 		(layer "F.Cu")
-		(at 143.07 109.3 -90)
+		(at 143.07 108.16 -90)
 		(descr "TO-220-3, Horizontal, RM 2.54mm, see https://www.vishay.com/docs/66542/to-220-1.pdf, generated with kicad-footprint-generator TO_SOT_THT_generate.py")
 		(tags "TO-220-3 Horizontal RM 2.54mm")
@@
 	)
 	(segment
-		(start 145.1 109.81)
-		(end 145.1 108)
-		(width 0.2)
-		(layer "F.Cu")
-		(net 6)
-	)
-	(segment
 		(start 187.21 106.215)
 		(end 184.15 109.275)
@@
 	)
 	(segment
-		(start 182.849 110.576)
-		(end 184.15 109.275)
+		(start 151.201 104.601)
+		(end 149.9 103.3)
 		(width 0.2)
 		(layer "F.Cu")
@@
 	)
 	(segment
-		(start 149.9 103.3)
-		(end 155.499 108.899)
+		(start 182.543917 110.881083)
+		(end 181.001 110.881083)
 		(width 0.2)
 		(layer "F.Cu")
@@
 	)
 	(segment
-		(start 180.695917 110.576)
-		(end 182.849 110.576)
+		(start 181.001 110.881083)
+		(end 174.720917 104.601)
 		(width 0.2)
 		(layer "F.Cu")
@@
 	)
 	(segment
-		(start 187.21 102.5)
-		(end 187.21 106.215)
+		(start 143.07 110.7)
+		(end 149.9 103.87)
 		(width 0.2)
 		(layer "F.Cu")
@@
 	)
 	(segment
-		(start 179.018917 108.899)
-		(end 180.695917 110.576)
+		(start 174.720917 104.601)
+		(end 151.201 104.601)
 		(width 0.2)
 		(layer "F.Cu")
@@
 	)
 	(segment
-		(start 145.1 108)
-		(end 149.8 103.3)
+		(start 187.21 102.5)
+		(end 187.21 106.215)
 		(width 0.2)
 		(layer "F.Cu")
@@
 	)
 	(segment
-		(start 143.07 111.84)
-		(end 145.1 109.81)
+		(start 184.15 109.275)
+		(end 182.543917 110.881083)
 		(width 0.2)
 		(layer "F.Cu")
@@
 	)
 	(segment
-		(start 155.499 108.899)
-		(end 179.018917 108.899)
+		(start 149.9 103.87)
+		(end 149.9 103.3)
 		(width 0.2)
 		(layer "F.Cu")
@@
 	)
 	(segment
-		(start 131.176 109.551)
-		(end 142.819 109.551)
-		(width 0.2)
-		(layer "F.Cu")
-		(net 7)
-	)
-	(segment
-		(start 143.07 102.16)
+		(start 136.575 101.6)
 		(end 142.51 101.6)
 		(width 0.2)
@@
 	)
 	(segment
-		(start 142.819 109.551)
-		(end 143.07 109.3)
+		(start 143.07 108.16)
+		(end 143.07 102.16)
 		(width 0.2)
 		(layer "F.Cu")
@@
 	)
 	(segment
-		(start 143.07 109.3)
-		(end 143.07 102.16)
+		(start 143.07 102.16)
+		(end 142.51 101.6)
 		(width 0.2)
 		(layer "F.Cu")
@@
 	(segment
 		(start 129.9 108.275)
-		(end 131.176 109.551)
+		(end 136.575 101.6)
 		(width 0.2)
 		(layer "F.Cu")
