File: schematics/spider_dropper/spider_dropper.kicad_pcb (KiCad board)
At the start: 2 copper layers, 80 x 20 mm, 10 parts, among them J1 JST_XH_3, J2 PJ-044AH, J3 JST_XH_2, Q1 IRLZ34N, SW1 ZX40E20C01

Commit message: Final Revision E PCB heading to PCBWay for Make & Take boards.
Routing:
- net GND: vias 0 -> 2
- added copper zone on F.Cu, net GND
- removed copper zone on F.Cu, net (none)
Other:
- board text added: "Rev. E - 2026"
- board text removed: "Rev. E - 2025"
