File: schematics/spider_dropper/spider_dropper.kicad_sch (KiCad schematic)
At the start: 18 parts, among them J1 JST_XH_3, J2 PJ-044AH, J3 JST_XH_2, Q1 IRLZ34N, SW1 ZX40E20C01

Commit message: Changed the diode footprint to a DO-41.
The leads of the 1N4001 diodes I have barely fit into the holes for the
default footprint.  Datasheet suggests DO-41 is the correct package,
and KiCad has a footprint for that with the same spacing but larger
holes.
Parts:
- D1: footprint Diode_THT:D_A-405_P7.62mm_Horizontal -> Diode_THT:D_DO-41_SOD81_P7.62mm_Horizontal
Changed lines of the file:
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@@
 	(title_block
 		(title "Slightly Smarter Spider Dropper")
-		(date "2025-09-11")
+		(date "2025-09-21")
 		(rev "E")
 		(company "Adrian McCarthy")
@@
 			)
 		)
-		(property "Footprint" "Diode_THT:D_A-405_P7.62mm_Horizontal"
+		(property "Footprint" "Diode_THT:D_DO-41_SOD81_P7.62mm_Horizontal"
 			(at 140.97 64.77 0)
 			(effects

Commit message: Switched to smaller, cheaper signal diode.
The 1N4001 was overkill for the motor flyback.  The 1N4148 is a common
signal diode that fits the space a little better.

Also nudged the connector for the motor controller to help my fat
fingers access it.
Parts:
- D1: value 1N4001 -> 1N4148; footprint Diode_THT:D_DO-41_SOD81_P7.62mm_Horizontal -> Diode_THT:D_DO-35_SOD27_P7.62mm_Horizontal
Changed lines of the file:
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@@
 	(title_block
 		(title "Slightly Smarter Spider Dropper")
-		(date "2025-09-21")
+		(date "2025-09-27")
 		(rev "E")
 		(company "Adrian McCarthy")
@@
 			)
 		)
-		(property "Value" "1N4001"
+		(property "Value" "1N4148"
 			(at 143.002 65.9821 90)
 			(effects
@@
 			)
 		)
-		(property "Footprint" "Diode_THT:D_DO-41_SOD81_P7.62mm_Horizontal"
+		(property "Footprint" "Diode_THT:D_DO-35_SOD27_P7.62mm_Horizontal"
 			(at 140.97 64.77 0)
 			(effects

Commit message: Reverted change to the diode.  Back to 1N4001.
Parts:
- D1: value 1N4148 -> 1N4001; footprint Diode_THT:D_DO-35_SOD27_P7.62mm_Horizontal -> Diode_THT:D_DO-41_SOD81_P7.62mm_Horizontal
Changed lines of the file:
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@@
 	(title_block
 		(title "Slightly Smarter Spider Dropper")
-		(date "2025-09-27")
+		(date "2025-10-14")
 		(rev "E")
 		(company "Adrian McCarthy")
@@
 			)
 		)
-		(property "Value" "1N4148"
+		(property "Value" "1N4001"
 			(at 143.002 65.9821 90)
 			(effects
@@
 			)
 		)
-		(property "Footprint" "Diode_THT:D_DO-35_SOD27_P7.62mm_Horizontal"
+		(property "Footprint" "Diode_THT:D_DO-41_SOD81_P7.62mm_Horizontal"
 			(at 140.97 64.77 0)
 			(effects
